File: hardware/board/U_depot.sch (KiCad schematic (older format))
At the start: 19 parts

Commit message: parts addded
Parts:
- C? (x2): value C -> 10 uF
- D?: value ZENER -> BZV55-B3V6,115
- D? (x2): value D_Schottky -> CUS08F30,H3F
- Q?: value Q_NPN_BCE -> PBHV8118T,215
- Q? (x2): value Q_NMOS_DGS -> NTR5103NT1G
- R?: value R -> 47
- R?: value R -> 100k
- gave numbers to parts that had none: 1
Changed lines of the file:
@@
 P 3200 3950
 F 0 "R?" V 3280 3950 50  0000 C CNN
-F 1 "R" V 3200 3950 50  0000 C CNN
+F 1 "47" V 3200 3950 50  0000 C CNN
 F 2 "" V 3130 3950 50  0000 C CNN
 F 3 "" H 3200 3950 50  0000 C CNN
@@
 P 3200 4450
 F 0 "D?" H 3200 4550 50  0000 C CNN
-F 1 "ZENER" H 3200 4350 50  0000 C CNN
+F 1 "BZV55-B3V6,115" H 3200 4350 50  0000 C CNN
 F 2 "" H 3200 4450 50  0000 C CNN
 F 3 "" H 3200 4450 50  0000 C CNN
@@
 P 5800 4000
 F 0 "Q?" H 6100 4050 50  0000 R CNN
-F 1 "Q_NPN_BCE" H 6400 3950 50  0000 R CNN
+F 1 "PBHV8118T,215" H 6400 3950 50  0000 R CNN
 F 2 "" H 6000 4100 50  0000 C CNN
 F 3 "" H 5800 4000 50  0000 C CNN
@@
 $EndComp
 $Comp
-L C C?
+L C 8.83mF
 U 1 1 5883D158
 P 6050 4500
-F 0 "C?" H 6075 4600 50  0000 L CNN
+F 0 "8.83mF" H 6075 4600 50  0000 L CNN
 F 1 "C" H 6075 4400 50  0000 L CNN
 F 2 "" H 6088 4350 50  0000 C CNN
@@
 P 5550 4150
 F 0 "R?" V 5630 4150 50  0000 C CNN
-F 1 "R" V 5550 4150 50  0000 C CNN
+F 1 "100k" V 5550 4150 50  0000 C CNN
 F 2 "" V 5480 4150 50  0000 C CNN
 F 3 "" H 5550 4150 50  0000 C CNN
@@
 P 6500 4550
 F 0 "Q?" H 6700 4600 50  0000 L CNN
-F 1 "Q_NMOS_DGS" H 6700 4500 50  0000 L CNN
+F 1 "NTR5103NT1G" H 6700 4500 50  0000 L CNN
 F 2 "" H 6700 4650 50  0000 C CNN
 F 3 "" H 6500 4550 50  0000 C CNN
@@
 P 6850 3700
 F 0 "D?" H 6850 3800 50  0000 C CNN
-F 1 "D_Schottky" H 6850 3600 50  0000 C CNN
+F 1 "CUS08F30,H3F" H 6850 3600 50  0000 C CNN
 F 2 "" H 6850 3700 50  0000 C CNN
 F 3 "" H 6850 3700 50  0000 C CNN
@@
 P 7150 3850
 F 0 "C?" H 7175 3950 50  0000 L CNN
-F 1 "C" H 7175 3750 50  0000 L CNN
+F 1 "10 uF" H 7175 3750 50  0000 L CNN
 F 2 "" H 7188 3700 50  0000 C CNN
 F 3 "" H 7150 3850 50  0000 C CNN
@@
 P 7450 3700
 F 0 "D?" H 7450 3800 50  0000 C CNN
-F 1 "D_Schottky" H 7450 3600 50  0000 C CNN
+F 1 "CUS08F30,H3F" H 7450 3600 50  0000 C CNN
 F 2 "" H 7450 3700 50  0000 C CNN
 F 3 "" H 7450 3700 50  0000 C CNN
@@
 P 7750 3850
 F 0 "C?" H 7775 3950 50  0000 L CNN
-F 1 "C" H 7775 3750 50  0000 L CNN
+F 1 "10 uF" H 7775 3750 50  0000 L CNN
 F 2 "" H 7788 3700 50  0000 C CNN
 F 3 "" H 7750 3850 50  0000 C CNN
@@
 P 8600 3900
 F 0 "Q?" H 8800 3950 50  0000 L CNN
-F 1 "Q_NMOS_DGS" H 8800 3850 50  0000 L CNN
+F 1 "NTR5103NT1G" H 8800 3850 50  0000 L CNN
 F 2 "" H 8800 4000 50  0000 C CNN
 F 3 "" H 8600 3900 50  0000 C CNN

Commit message: finish with footprints
Parts:
- removed P?: CONN_01X02, symbol CONN_01X02
- added C3: 4.5mF, Capacitors_THT:CP_Radial_D18.0mm_P7.50mm, symbol C
- added P1: CAM, Pin_Headers:Pin_Header_Angled_1x04_Pitch2.54mm, symbol CONN_01X04
- added P2, P3: CONN_01X14, Pin_Headers:Pin_Header_Angled_1x14_Pitch2.54mm, symbol CONN_01X14
- C1, C2: renamed from C?; footprint (none) -> Capacitors_THT:CP_Radial_D5.0mm_P2.00mm
- C4: renamed from 8.83mF; value C -> 4.5mF; footprint (none) -> Capacitors_THT:CP_Radial_D18.0mm_P7.50mm
- D1, D3: renamed from D?; footprint (none) -> Diodes_SMD:D_SMC_Standard
- D2: renamed from D?; footprint (none) -> Diodes_SMD:D_SCD80_HandSoldering
- D4: renamed from D?; footprint (none) -> Diodes_SMD:D_SOD-323
- D5: renamed from D?; footprint (none) -> Diodes_SMD:D_SOD-323_HandSoldering
- Q1, Q2, Q3: renamed from Q?; footprint (none) -> TO_SOT_Packages_SMD:SOT-23
- R1, R2, R3: renamed from R?; footprint (none) -> Resistors_SMD:R_0603_HandSoldering
- R4, R5, R6: renamed from R?; footprint (none) -> Resistors_SMD:R_0805_HandSoldering
- U1: renamed from U?; footprint SC70-5 -> TO_SOT_Packages_SMD:SOT-23-5_HandSoldering
Connections:
- net 3.3V: now also P3.3 (P3)
- net GND: now also C3.2, P1.3 (P3), P2.1 (P1)
- net at D3.2 (A), Q1.3 (E), Q2.1 (D): now also C3.1; no longer C4.1
- net at Q2.3 (S): now also P1.4 (P4)
- new net AGND: P3.2 (P2)
- new net RX1: P2.2 (P2)
- new net RX2: P2.11 (P11)
- new net RX3: P2.9 (P9)
- new net Rx: P1.2 (P2)
- new net SCK: P3.14 (P14)
- new net SCL: P3.8 (P8)
- new net SDA: P3.9 (P9)
- new net TX1: P2.3 (P3)
- new net TX2: P2.12 (P12)
- new net TX3: P2.10 (P10)
- new net Tx: P1.1 (P1)
- new net Vin: P3.1 (P1)
Other:
- moved on the sheet: C4

Commit message: started designing board
Parts:
- P2, P3: value CONN_01X14 -> TEENSY 3.2; footprint Pin_Headers:Pin_Header_Angled_1x14_Pitch2.54mm -> Pin_Headers:Pin_Header_Straight_1x14_Pitch2.54mm
Changed lines of the file:
@@
 P 8800 5650
 F 0 "P2" H 8800 6400 50  0000 C CNN
-F 1 "CONN_01X14" V 8900 5650 50  0000 C CNN
-F 2 "Pin_Headers:Pin_Header_Angled_1x14_Pitch2.54mm" H 8800 5650 50  0001 C CNN
+F 1 "TEENSY 3.2" V 8900 5650 50  0000 C CNN
+F 2 "Pin_Headers:Pin_Header_Straight_1x14_Pitch2.54mm" H 8800 5650 50  0001 C CNN
 F 3 "" H 8800 5650 50  0000 C CNN
 	1    8800 5650
@@
 P 9200 5650
 F 0 "P3" H 9200 6400 50  0000 C CNN
-F 1 "CONN_01X14" V 9300 5650 50  0000 C CNN
-F 2 "Pin_Headers:Pin_Header_Angled_1x14_Pitch2.54mm" H 9200 5650 50  0001 C CNN
+F 1 "TEENSY 3.2" V 9300 5650 50  0000 C CNN
+F 2 "Pin_Headers:Pin_Header_Straight_1x14_Pitch2.54mm" H 9200 5650 50  0001 C CNN
 F 3 "" H 9200 5650 50  0000 C CNN
 	1    9200 5650

Commit message: updated schottky diode footprint
Parts:
- D1, D3: footprint Diodes_SMD:D_SMC_Standard -> Diodes_SMD:D_SMB_Handsoldering
Changed lines of the file:
@@
 F 0 "D1" H 2750 3800 50  0000 C CNN
 F 1 "LSM115JE3/TR13" H 2750 3600 50  0000 C CNN
-F 2 "Diodes_SMD:D_SMC_Standard" H 2750 3700 50  0001 C CNN
+F 2 "Diodes_SMD:D_SMB_Handsoldering" H 2750 3700 50  0001 C CNN
 F 3 "" H 2750 3700 50  0000 C CNN
 	1    2750 3700
@@
 F 0 "D3" H 6650 4050 50  0000 C CNN
 F 1 "LSM115JE3/TR13" H 6650 3850 50  0000 C CNN
-F 2 "Diodes_SMD:D_SMC_Standard" H 6650 3950 50  0001 C CNN
+F 2 "Diodes_SMD:D_SMB_Handsoldering" H 6650 3950 50  0001 C CNN
 F 3 "" H 6650 3950 50  0000 C CNN
 F 4 "LSM115JE3/TR13" H 6650 3950 60  0001 C CNN "Part Number"
